Commit message: Made the blue turtle purple. Go Cats

File: nuturtle_description/urdf/common_properties.xacro (robot description, xacro)
@@ -32,3 +32,6 @@
     <color rgba="1.0 1.0 1.0 1.0"/>
   </material>
+  <material name="nu_purple">
+    <color rgba="0.3 0.16 0.52 1.0"/>
+  </material>
 </robot>
